File: kicad_docs/power_supply.sch (KiCad schematic (older format))
At the start: 28 parts, among them J6 iec_power_entry, SW1 power_on, T1 power_transformer, U1 5879, U2 6SN7, U3 6SN7, U5 6V6, U6 6V6

Commit message: add approximate voltages
Other:
- note added: "-55 VDC"
- note added: "120 VAC in"
- note added: "22 VAC"
- note added: "290 VAC"
- note added: "300 VDC"
- note added: "310 VDC"
- note added: "330 VDC"
- note added: "385 VDC"
- note added: "390 VDC"
- note added: "6.3 VAC"
- note added: "All voltages approximate"
- note added: "approximately\n350mA @ idle\n650mA @ max"
- note removed: "120VAC in"
- note removed: "6.3VAC"
- note removed: "???VAC"
- moved on the sheet: C23, C27, C28, L1, R54, R55, R56
Changed lines of the file:
@@
 Wire Wire Line
 	4500 2150 4500 2250
-Text GLabel 6400 1350 2    50   Output ~ 0
+Text GLabel 6200 1350 2    50   Output ~ 0
 B+_1
 $Comp
 L Device:L L1
 U 1 1 610B3013
-P 6750 1750
-F 0 "L1" V 6940 1750 50  0000 C CNN
-F 1 "choke" V 6849 1750 50  0000 C CNN
-F 2 "" H 6750 1750 50  0001 C CNN
-F 3 "~" H 6750 1750 50  0001 C CNN
-	1    6750 1750
+P 6550 1750
+F 0 "L1" V 6740 1750 50  0000 C CNN
+F 1 "choke" V 6649 1750 50  0000 C CNN
+F 2 "" H 6550 1750 50  0001 C CNN
+F 3 "~" H 6550 1750 50  0001 C CNN
+	1    6550 1750
 	0    -1   -1   0
 $EndComp
@@
 L Device:CP1 C23
 U 1 1 610B483F
-P 7300 2150
-F 0 "C23" H 7415 2196 50  0000 L CNN
-F 1 "47u 500v" H 7415 2105 50  0000 L CNN
-F 2 "" H 7300 2150 50  0001 C CNN
-F 3 "~" H 7300 2150 50  0001 C CNN
-	1    7300 2150
-	1    0    0    -1
-$EndComp
-Wire Wire Line
-	5950 1750 6250 1750
+P 7200 2150
+F 0 "C23" H 7315 2196 50  0000 L CNN
+F 1 "47u 500v" H 7315 2105 50  0000 L CNN
+F 2 "" H 7200 2150 50  0001 C CNN
+F 3 "~" H 7200 2150 50  0001 C CNN
+	1    7200 2150
+	1    0    0    -1
+$EndComp
+Wire Wire Line
+	5950 1750 6050 1750
 Connection ~ 5950 1750
 Wire Wire Line
-	6400 1350 6250 1350
-Wire Wire Line
-	6250 1350 6250 1750
-Connection ~ 6250 1750
-Wire Wire Line
-	6250 1750 6600 1750
-Wire Wire Line
-	7300 2000 7300 1750
-Wire Wire Line
-	7300 1750 7150 1750
+	6200 1350 6050 1350
+Wire Wire Line
+	6050 1350 6050 1750
+Connection ~ 6050 1750
+Wire Wire Line
+	6050 1750 6400 1750
+Wire Wire Line
+	7200 2000 7200 1750
+Wire Wire Line
+	7200 1750 7050 1750
 $Comp
 L Device:R R54
 U 1 1 610BF1DC
-P 7750 1750
-F 0 "R54" V 7543 1750 50  0000 C CNN
-F 1 "3k 5W" V 7634 1750 50  0000 C CNN
-F 2 "" V 7680 1750 50  0001 C CNN
-F 3 "~" H 7750 1750 50  0001 C CNN
-	1    7750 1750
+P 7700 1750
+F 0 "R54" V 7493 1750 50  0000 C CNN
+F 1 "3k 5W" V 7584 1750 50  0000 C CNN
+F 2 "" V 7630 1750 50  0001 C CNN
+F 3 "~" H 7700 1750 50  0001 C CNN
+	1    7700 1750
 	0    1    1    0
 $EndComp
@@
 L Device:R R55
 U 1 1 610C3F28
-P 8650 1750
-F 0 "R55" V 8443 1750 50  0000 C CNN
-F 1 "2k7 1W" V 8534 1750 50  0000 C CNN
-F 2 "" V 8580 1750 50  0001 C CNN
-F 3 "~" H 8650 1750 50  0001 C CNN
-	1    8650 1750
+P 8750 1750
+F 0 "R55" V 8543 1750 50  0000 C CNN
+F 1 "2k7 1W" V 8634 1750 50  0000 C CNN
+F 2 "" V 8680 1750 50  0001 C CNN
+F 3 "~" H 8750 1750 50  0001 C CNN
+	1    8750 1750
 	0    1    1    0
 $EndComp
@@
 L Device:CP1 C27
 U 1 1 610C3F2E
-P 9150 2150
-F 0 "C27" H 9265 2196 50  0000 L CNN
-F 1 "22u 450v" H 9265 2105 50  0000 L CNN
-F 2 "" H 9150 2150 50  0001 C CNN
-F 3 "~" H 9150 2150 50  0001 C CNN
-	1    9150 2150
+P 9300 2150
+F 0 "C27" H 9415 2196 50  0000 L CNN
+F 1 "22u 450v" H 9415 2105 50  0000 L CNN
+F 2 "" H 9300 2150 50  0001 C CNN
+F 3 "~" H 9300 2150 50  0001 C CNN
+	1    9300 2150
 	1    0    0    -1
 $EndComp
@@
 L Device:R R56
 U 1 1 610C5FC4
-P 9550 1750
-F 0 "R56" V 9343 1750 50  0000 C CNN
-F 1 "2k2 1W" V 9434 1750 50  0000 C CNN
-F 2 "" V 9480 1750 50  0001 C CNN
-F 3 "~" H 9550 1750 50  0001 C CNN
-	1    9550 1750
+P 9800 1750
+F 0 "R56" V 9593 1750 50  0000 C CNN
+F 1 "2k2 1W" V 9684 1750 50  0000 C CNN
+F 2 "" V 9730 1750 50  0001 C CNN
+F 3 "~" H 9800 1750 50  0001 C CNN
+	1    9800 1750
 	0    1    1    0
 $EndComp
@@
 L Device:CP1 C28
 U 1 1 610C5FCA
-P 10050 2150
-F 0 "C28" H 10165 2196 50  0000 L CNN
-F 1 "22u 450v" H 10165 2105 50  0000 L CNN
-F 2 "" H 10050 2150 50  0001 C CNN
-F 3 "~" H 10050 2150 50  0001 C CNN
-	1    10050 2150
-	1    0    0    -1
-$EndComp
-Wire Wire Line
-	7600 1750 7300 1750
-Connection ~ 7300 1750
-Wire Wire Line
-	7900 1750 8150 1750
-Wire Wire Line
-	8800 1750 9050 1750
-Wire Wire Line
-	9700 1750 9950 1750
-Wire Wire Line
-	10050 1750 10050 2000
-Wire Wire Line
-	9150 2000 9150 1750
-Connection ~ 9150 1750
-Wire Wire Line
-	9150 1750 9400 1750
+P 10350 2150
+F 0 "C28" H 10465 2196 50  0000 L CNN
+F 1 "22u 450v" H 10465 2105 50  0000 L CNN
+F 2 "" H 10350 2150 50  0001 C CNN
+F 3 "~" H 10350 2150 50  0001 C CNN
+	1    10350 2150
+	1    0    0    -1
+$EndComp
+Wire Wire Line
+	7550 1750 7200 1750
+Connection ~ 7200 1750
+Wire Wire Line
+	7850 1750 8150 1750
+Wire Wire Line
+	8900 1750 9200 1750
+Wire Wire Line
+	9950 1750 10250 1750
+Wire Wire Line
+	10350 1750 10350 2000
+Wire Wire Line
+	9300 2000 9300 1750
+Connection ~ 9300 1750
+Wire Wire Line
+	9300 1750 9650 1750
 Wire Wire Line
 	8250 2000 8250 1750
 Connection ~ 8250 1750
 Wire Wire Line
-	8250 1750 8500 1750
-Wire Wire Line
-	10050 2300 10050 2550
-Wire Wire Line
-	10050 2550 9150 2550
-Wire Wire Line
-	7300 2550 7300 2300
+	8250 1750 8600 1750
+Wire Wire Line
+	10350 2300 10350 2550
+Wire Wire Line
+	10350 2550 9300 2550
+Wire Wire Line
+	7200 2550 7200 2300
 Wire Wire Line
 	8250 2300 8250 2550
 Connection ~ 8250 2550
 Wire Wire Line
-	8250 2550 7300 2550
-Wire Wire Line
-	9150 2300 9150 2550
-Connection ~ 9150 2550
-Wire Wire Line
-	9150 2550 8250 2550
-Text GLabel 7300 1350 2    50   Output ~ 0
+	8250 2550 7200 2550
+Wire Wire Line
+	9300 2300 9300 2550
+Connection ~ 9300 2550
+Wire Wire Line
+	9300 2550 8250 2550
+Text GLabel 7200 1350 2    50   Output ~ 0
 B+_2
 Wire Wire Line
-	7300 1350 7150 1350
-Wire Wire Line
-	7150 1350 7150 1750
+	7200 1350 7050 1350
+Wire Wire Line
+	7050 1350 7050 1750
 Text GLabel 8300 1350 2    50   Output ~ 0
 B+_3
@@
 Wire Wire Line
 	8150 1350 8150 1750
-Text GLabel 9200 1350 2    50   Output ~ 0
+Text GLabel 9350 1350 2    50   Output ~ 0
 B+_4
 Wire Wire Line
-	9200 1350 9050 1350
-Wire Wire Line
-	9050 1350 9050 1750
-Text GLabel 10100 1350 2    50   Output ~ 0
+	9350 1350 9200 1350
+Wire Wire Line
+	9200 1350 9200 1750
+Text GLabel 10400 1350 2    50   Output ~ 0
 B+_5
 Wire Wire Line
-	10100 1350 9950 1350
-Wire Wire Line
-	9950 1350 9950 1750
-Connection ~ 9950 1750
-Wire Wire Line
-	9950 1750 10050 1750
-Connection ~ 9050 1750
-Wire Wire Line
-	9050 1750 9150 1750
+	10400 1350 10250 1350
+Wire Wire Line
+	10250 1350 10250 1750
+Connection ~ 10250 1750
+Wire Wire Line
+	10250 1750 10350 1750
+Connection ~ 9200 1750
+Wire Wire Line
+	9200 1750 9300 1750
 Connection ~ 8150 1750
 Wire Wire Line
@@
 	1    0    0    -1
 $EndComp
-Connection ~ 7300 2550
-Connection ~ 7150 1750
-Wire Wire Line
-	7150 1750 6900 1750
+Connection ~ 7200 2550
+Connection ~ 7050 1750
+Wire Wire Line
+	7050 1750 6700 1750
 $Comp
 L A200_custom_valves:6SN7 U2
@@
 	8200 4050 8200 3900
 Wire Wire Line
-	7300 2700 7300 2550
+	7200 2700 7200 2550
 $Comp
 L power:GND #PWR07
 U 1 1 61285A8B
-P 7300 2700
-F 0 "#PWR07" H 7300 2450 50  0001 C CNN
-F 1 "GND" H 7305 2527 50  0000 C CNN
-F 2 "" H 7300 2700 50  0001 C CNN
-F 3 "" H 7300 2700 50  0001 C CNN
-	1    7300 2700
+P 7200 2700
+F 0 "#PWR07" H 7200 2450 50  0001 C CNN
+F 1 "GND" H 7205 2527 50  0000 C CNN
+F 2 "" H 7200 2700 50  0001 C CNN
+F 3 "" H 7200 2700 50  0001 C CNN
+	1    7200 2700
 	1    0    0    -1
 $EndComp
@@
 U 1 1 6104DBEE
 P 1000 3050
-F 0 "J6" V 414 2992 50  0000 C CNN
+F 0 "J6" V 400 3050 50  0000 C CNN
 F 1 "iec_power_entry" V 505 2992 50  0000 C CNN
 F 2 "" V 1000 3050 50  0001 C CNN
@@
 	1600 3050 1350 3050
 Text Notes 3650 4050 0    118  ~ 0
-6.3VAC
+6.3 VAC
 Text Notes 3650 3550 0    118  ~ 0
-???VAC
+22 VAC
 Text Notes 3650 2900 0    118  ~ 0
-???VAC
-Text Notes 600  2350 0    118  ~ 0
-120VAC in
+290 VAC
+Text Notes 600  2050 0    118  ~ 0
+120 VAC in
+Text Notes 5950 1250 0    118  ~ 0
+390 VDC
+Text Notes 6950 1250 0    118  ~ 0
+385 VDC
+Text Notes 8050 1250 0    118  ~ 0
+330 VDC
+Text Notes 9100 1250 0    118  ~ 0
+310 VDC
+Text Notes 10150 1250 0    118  ~ 0
+300 VDC
+Text Notes 7900 4950 0    118  ~ 0
+-55 VDC
+Text Notes 750  2350 0    50   ~ 0
+approximately\n350mA @ idle\n650mA @ max
+Text Notes 7400 6150 0    157  ~ 0
+All voltages approximate
 $EndSCHEMATC

Commit message: fix wrong tube number, reorder sheets
Parts:
- renumbered U5 to U4, U6 to U5
Changed lines of the file:
@@
 $EndComp
 $Comp
-L A200_custom_valves:6V6 U5
+L A200_custom_valves:6V6 U4
 U 2 1 611117DF
 P 4850 5850
-F 0 "U5" H 5078 5863 50  0000 L CNN
+F 0 "U4" H 5078 5863 50  0000 L CNN
 F 1 "6V6" H 5078 5772 50  0000 L CNN
 F 2 "octal" H 5150 5450 50  0001 C CNN
@@
 $EndComp
 $Comp
-L A200_custom_valves:6V6 U6
+L A200_custom_valves:6V6 U5
 U 2 1 61113A8C
 P 5600 5850
-F 0 "U6" H 5828 5863 50  0000 L CNN
+F 0 "U5" H 5828 5863 50  0000 L CNN
 F 1 "6V6" H 5828 5772 50  0000 L CNN
 F 2 "octal" H 5900 5450 50  0001 C CNN
